File: pcb/xbx-nrf-dongle/xbx-nrf-dongle.kicad_pcb (KiCad board)
At the start: 2 copper layers, 7 parts, among them J1 16P-USBC-RECEPTACLE, U1 MDBT50Q-1MV2, U2 USBLC6-2SC6, Y1 32.768kHz

Commit message: Rev1 positioning complete, pre-routing commit
Parts:
- added C1: 10uF, Capacitor_SMD:C_0805_2012Metric_Pad1.18x1.45mm_HandSolder, F.Cu at (78.5, 97.5)
- added C3: 10nF, Capacitor_SMD:C_0603_1608Metric_Pad1.08x0.95mm_HandSolder, F.Cu at (77.6, 100.9)
- added C4: 1uF, Capacitor_SMD:C_0603_1608Metric_Pad1.08x0.95mm_HandSolder, F.Cu at (70.4, 97.8)
- added C5: 10uF, Capacitor_SMD:C_0805_2012Metric_Pad1.18x1.45mm_HandSolder, F.Cu at (96.4, 85.1)
- added C6: 4.7uF, Capacitor_SMD:C_0805_2012Metric_Pad1.18x1.45mm_HandSolder, F.Cu at (98.0, 88.3)
- added C7: 9pF, Capacitor_SMD:C_0603_1608Metric_Pad1.08x0.95mm_HandSolder, F.Cu at (93.7, 78.2)
- added C8: 9pF, Capacitor_SMD:C_0603_1608Metric_Pad1.08x0.95mm_HandSolder, F.Cu at (93.5, 82.7)
- added D1: LED_BLUE, LED_SMD:LED_0603_1608Metric_Pad1.05x0.95mm_HandSolder, F.Cu at (84.5, 75.3)
- added D2: LED_GREEN, LED_SMD:LED_0603_1608Metric_Pad1.05x0.95mm_HandSolder, F.Cu at (114.5, 103.8)
- added D3: LED_GREEN, LED_SMD:LED_0603_1608Metric_Pad1.05x0.95mm_HandSolder, F.Cu at (114.5, 100.6)
- added D4: LED_GREEN, LED_SMD:LED_0603_1608Metric_Pad1.05x0.95mm_HandSolder, F.Cu at (114.5, 97.4)
- added D5: LED_GREEN, LED_SMD:LED_0603_1608Metric_Pad1.05x0.95mm_HandSolder, F.Cu at (114.5, 94.0)
- added D6: LED_RED, LED_SMD:LED_0603_1608Metric_Pad1.05x0.95mm_HandSolder, F.Cu at (85.0, 95.3)
- added H1: MountingHole, MountingHole:MountingHole_2.2mm_M2, F.Cu at (86.2, 64.5)
- added H2: MountingHole, MountingHole:MountingHole_2.2mm_M2, F.Cu at (121.2, 87.1)
- added H3: MountingHole, MountingHole:MountingHole_2.2mm_M2, F.Cu at (86.2, 109.5)
- added J1: SWD, Connector_JST:JST_SH_SM03B-SRSS-TB_1x03-1MP_P1.00mm_Horizontal, F.Cu at (102.9, 104.5)
- added J2: UART, Connector_JST:JST_SH_SM03B-SRSS-TB_1x03-1MP_P1.00mm_Horizontal, F.Cu at (94.4, 104.7)
- added JP1: SolderJumper_3_Open, Jumper:SolderJumper-3_P2.0mm_Open_TrianglePad1.0x1.5mm_NumberLabels, F.Cu at (89.7, 92.2)
- added R1: 10k, Resistor_SMD:R_0603_1608Metric_Pad0.98x0.95mm_HandSolder, F.Cu at (76.5, 77.8)
- added R10: 1k, Resistor_SMD:R_0603_1608Metric_Pad0.98x0.95mm_HandSolder, F.Cu at (110.6, 97.4)
- added R11: 1k, Resistor_SMD:R_0603_1608Metric_Pad0.98x0.95mm_HandSolder, F.Cu at (110.6, 94.0)
- added R12: 1k, Resistor_SMD:R_0603_1608Metric_Pad0.98x0.95mm_HandSolder, F.Cu at (88.8, 97.8)
- added R3: 10k, Resistor_SMD:R_0603_1608Metric_Pad0.98x0.95mm_HandSolder, F.Cu at (76.5, 70.8)
- added R4: 27R, Resistor_SMD:R_0603_1608Metric_Pad0.98x0.95mm_HandSolder, F.Cu at (80.7, 91.7)
- added R5: 27R, Resistor_SMD:R_0603_1608Metric_Pad0.98x0.95mm_HandSolder, F.Cu at (78.8, 91.7)
- added R7: 180R, Resistor_SMD:R_0603_1608Metric_Pad0.98x0.95mm_HandSolder, F.Cu at (80.5, 75.3)
- added R8: 1k, Resistor_SMD:R_0603_1608Metric_Pad0.98x0.95mm_HandSolder, F.Cu at (110.6, 103.8)
- added R9: 1k, Resistor_SMD:R_0603_1608Metric_Pad0.98x0.95mm_HandSolder, F.Cu at (110.6, 100.6)
- added SW1: SW_Push, Button_Switch_SMD:SW_SPST_B3U-1000P, F.Cu at (84.7, 100.3)
- added SW2: SW_Push, Button_Switch_SMD:SW_SPST_B3U-1000P, F.Cu at (84.7, 70.3)
- added SW3: SW_SPDT, sw-spdt-horizontal:SW_JS102011SAQN, F.Cu at (70.0, 74.2)
- added TP1: NRST, TestPoint:TestPoint_Pad_1.5x1.5mm, F.Cu at (93.5, 96.7)
- added TP10: 3v3, TestPoint:TestPoint_Pad_1.0x1.0mm, F.Cu at (103.9, 63.2)
- added TP11: VBUS, TestPoint:TestPoint_Pad_1.0x1.0mm, F.Cu at (69.5, 93.7)
- added TP12: AIN6, TestPoint:TestPoint_Pad_1.0x1.0mm, F.Cu at (98.4, 68.3)
- added TP13: AIN7, TestPoint:TestPoint_Pad_1.0x1.0mm, F.Cu at (103.8, 68.3)
- added TP14: P0.04, TestPoint:TestPoint_Pad_1.0x1.0mm, F.Cu at (93.0, 72.3)
- added TP15: P0.06, TestPoint:TestPoint_Pad_1.0x1.0mm, F.Cu at (103.8, 72.3)
- added TP16: P0.26, TestPoint:TestPoint_Pad_1.0x1.0mm, F.Cu at (98.4, 72.3)
- added TP17: P0.27, TestPoint:TestPoint_Pad_1.0x1.0mm, F.Cu at (93.0, 68.3)
- added TP2: VTREF, TestPoint:TestPoint_Pad_1.5x1.5mm, F.Cu at (106.1, 96.7)
- added TP3: SWO, TestPoint:TestPoint_Pad_1.5x1.5mm, F.Cu at (101.9, 96.7)
- added TP4: TIM, TestPoint:TestPoint_Pad_1.5x1.5mm, F.Cu at (97.7, 96.7)
- added TP5: GND, TestPoint:TestPoint_Pad_1.0x1.0mm, F.Cu at (95.2, 63.2)
- added TP6: GND, TestPoint:TestPoint_Pad_1.0x1.0mm, F.Cu at (91.8, 63.2)
- added TP7: GND, TestPoint:TestPoint_Pad_1.0x1.0mm, F.Cu at (98.6, 63.2)
- added TP8: 3v3, TestPoint:TestPoint_Pad_1.0x1.0mm, F.Cu at (110.7, 63.2)
- added TP9: 3v3, TestPoint:TestPoint_Pad_1.0x1.0mm, F.Cu at (107.3, 63.2)
- added U1: LDS3985M33R_SOT23, Package_TO_SOT_SMD:SOT-23-5, F.Cu at (74.4, 98.8)
- U3: renamed from U1; value MDBT50Q-1MV2 -> MDBT50Q-U1MV2
- Y1: footprint Crystal:Crystal_DS26_D2.0mm_L6.0mm_Horizontal -> Crystal:Crystal_SMD_3215-2Pin_3.2x1.5mm
- moved R2 48.7 mm to (79.8, 83.0)
- moved C2 42.6 mm to (84.7, 87.5)
- moved U2 42.5 mm to (79.8, 87.7), turned to -90 degrees
- moved R6 42.1 mm to (74.5, 92.7)
- moved J3 41.8 mm to (70.0, 86.0)
- moved Y1 29.2 mm to (96.6, 80.5), turned to 90 degrees
- moved U3 28.5 mm to (107.4, 83.4)
- renumbered C1 to C2, J1 to J3, R1 to R2, R2 to R6
Connections:
- net /D+_EXT renamed /EXT_D+
- net /D-_EXT renamed /EXT_D-
- U2 pad 4: /D- -> Net-(R5-Pad1)
- U2 pad 6: /D+ -> Net-(R4-Pad2)
- U3 pad 10: unconnected-(U1-P0.29-Pad10) -> /PWR_LED
- U3 pad 11: unconnected-(U1-P0.02-Pad11) -> /PAIR_LED
- U3 pad 12: unconnected-(U1-P0.31-Pad12) -> /AIN7
- U3 pad 14: unconnected-(U1-P0.30-Pad14) -> /AIN6
- U3 pad 16: unconnected-(U1-P0.27-Pad16) -> /P0.27
- U3 pad 19: unconnected-(U1-P0.26-Pad19) -> /P0.26
- U3 pad 20: unconnected-(U1-P0.04-Pad20) -> /P0.04
- U3 pad 22: unconnected-(U1-P0.06-Pad22) -> /P0.06
- U3 pad 28: unconnected-(U1-VDD-Pad28) -> +3V3
- U3 pad 30: unconnected-(U1-VDDH-Pad30) -> +3V3
- U3 pad 4: unconnected-(U1-P1.11-Pad4) -> /MODE_SW
- U3 pad 40: unconnected-(U1-P0.18-Pad40) -> /NRST
- U3 pad 41: unconnected-(U1-P0.17-Pad41) -> /TIMING_PIN
- U3 pad 43: unconnected-(U1-P0.21-Pad43) -> /DBG_TX
- U3 pad 44: unconnected-(U1-P0.20-Pad44) -> /DBG_RX
- U3 pad 47: unconnected-(U1-P1.00-Pad47) -> /SWO
- U3 pad 5: unconnected-(U1-P1.12-Pad5) -> /PAIR_SW
- U3 pad 51: unconnected-(U1-SWDIO-Pad51) -> /SWDIO
- U3 pad 53: unconnected-(U1-SWDCLK-Pad53) -> /SWCLK
- U3 pad 6: unconnected-(U1-P1.13-Pad6) -> /P1_LED
- U3 pad 7: unconnected-(U1-P1.14-Pad7) -> /P2_LED
- U3 pad 8: unconnected-(U1-P1.15-Pad8) -> /P3_LED
- U3 pad 9: unconnected-(U1-P0.03-Pad9) -> /P4_LED
Routing:
- net GND: track 0.00 -> 12.1 mm, vias 0 -> 7
- net /EXT_D+: track 0.00 -> 10.3 mm
- net /EXT_D-: track 0.00 -> 9.24 mm
- net Net-(U3-P0.01): track 0.00 -> 6.54 mm
- net Net-(U3-P0.00): track 0.00 -> 6.54 mm
- net +3V3: track 0.00 -> 5.59 mm, vias 0 -> 1
- net VBUS: track 0.00 -> 2.34 mm
Other:
- board outline added: 59.8 x 82.3 mm
- board text added: "3v3"
- board text added: "GND"

Commit message: Change board shape, reposition components. Pre-routing commit
Parts:
- removed the C4 at (70.4, 97.8)
- removed the H2 at (121.2, 87.1)
- removed the R3 at (76.5, 70.8)
- R2, TP1, TP10, TP2, TP3, TP4, TP5, TP6, TP7, TP8, TP9: moved to B.Cu
- R5: renamed from R6; moved to B.Cu
- moved C3 31.1 mm to (89.0, 72.0), turned to 0 degrees
- moved TP2 30.8 mm to (75.8, 102.2), turned to -90 degrees
- moved J1 30.6 mm to (72.3, 104.1), turned to -90 degrees
- moved D5 27.7 mm to (88.7, 104.0), turned to -90 degrees
- moved C1 27.4 mm to (85.6, 71.0), turned to 90 degrees
- moved U1 26.8 mm to (86.9, 75.2), turned to 90 degrees
- moved TP4 26.6 mm to (71.7, 102.3), turned to -90 degrees
- moved TP3 26.1 mm to (75.8, 98.0), turned to -90 degrees
- moved R10 26.0 mm to (88.7, 107.9), turned to 90 degrees
- moved J3 23.6 mm to (72.3, 96.4), turned to -90 degrees
- moved D4 23.4 mm to (92.1, 104.0), turned to -90 degrees
- moved TP1 21.9 mm to (71.7, 98.1), turned to -90 degrees
- moved R9 21.3 mm to (92.1, 107.9), turned to 90 degrees
- moved TP5 19.7 mm to (75.6, 65.5)
- moved TP6 19.7 mm to (72.2, 65.5)
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- renumbered C5 to C4, C6 to C5, C7 to C6, C8 to C7, H3 to H2, J3 to J2, J2 to J3, R11 to R10, R12 to R11, R4 to R3, R5 to R4, R7 to R6, R8 to R7, R9 to R8, R10 to R9
Connections:
- net Net-(U3-P0.00) renamed /XL1
- net Net-(U3-P0.01) renamed /XL2
- R1 pad 1: +3V3 -> GND
- R3 pad 1: /D+ -> /D-
- R4 pad 2: /D- -> /D+
- SW3 pad 1: Net-(R3-Pad1) -> unconnected-(SW3-Pad1)
- U2 pad 1: /EXT_D+ -> /EXT_D-
- U2 pad 3: /EXT_D- -> /EXT_D+
Routing:
- net VBUS: track 2.34 -> 19.6 mm
- net GND: track 12.1 -> 1.71 mm, vias 7 -> 33
- net /D+: track 0.00 -> 6.80 mm
- net /D-: track 0.00 -> 6.80 mm
- net /EXT_D+: track 10.3 -> 6.59 mm
- net Net-(J2-CC1): track 0.00 -> 2.99 mm, vias 0 -> 1
- net Net-(J2-CC2): track 0.00 -> 2.50 mm, vias 0 -> 1
- net Net-(R4-Pad1): track 0.00 -> 2.24 mm
- net Net-(R3-Pad2): track 0.00 -> 2.23 mm
- net /EXT_D-: track 9.24 -> 8.09 mm
- net +3V3: track 5.59 -> 4.90 mm, vias 1 -> 0
- net /XL1: track 6.54 -> 7.07 mm
- added copper zone on B.Cu, net GND
- added copper zone on F.Cu, net GND
Other:
- board size 59.8 x 82.3 mm -> 35 x 50 mm
- board text added: "ANTENNA ZONE"

Commit message: Dongle PCB Rev1 complete
Parts:
- J2: footprint usbc-16p-receptacle-amphenol:USB_C_Receptacle_16P_Amphenol_10155435-00011LF -> xbx-nrf-lib:USB_C_Receptacle_16P_Amphenol_10155435-00011LF
- JP1: footprint Jumper:SolderJumper-3_P2.0mm_Open_TrianglePad1.0x1.5mm_NumberLabels -> xbx-nrf-lib:SolderJumper-3_P2.0mm_Open_TrianglePad1.0x1.5mm_NumberLabels
- R1: value 10k -> 1k
- TP1, TP2, TP3, TP4: footprint TestPoint:TestPoint_Pad_1.5x1.5mm -> xbx-nrf-lib:TestPoint_Pad_1.5x1.5mm-NoSilkscreen
- TP10, TP11, TP12, TP13, TP14, TP15, TP16, TP17, TP5, TP6, TP7, TP8, TP9: footprint TestPoint:TestPoint_Pad_1.0x1.0mm -> xbx-nrf-lib:TestPoint_Pad_1.0x1.0mm-NoSilkscreen
- U3: footprint RF_Module:Raytac_MDBT50Q -> xbx-nrf-lib:Raytac_MDBT50Q
- Y1: footprint Crystal:Crystal_SMD_3215-2Pin_3.2x1.5mm -> xbx-nrf-lib:Crystal_SMD_3215-2Pin_3.2x1.5mm
- moved D5 31.2 mm to (106.2, 78.2)
- moved R10 31.2 mm to (106.2, 82.1)
- moved TP14 28.2 mm to (104.6, 47.3)
- moved D4 28.0 mm to (103.0, 78.2)
- moved R9 28.0 mm to (103.0, 82.1)
- moved H1 27.4 mm to (91.4, 40.7)
- moved J3 26.9 mm to (80.0, 70.6)
- moved TP3 26.9 mm to (83.5, 72.2)
- moved C1 26.9 mm to (93.3, 45.2)
- moved C2 26.9 mm to (85.6, 63.9)
- moved R3 26.9 mm to (91.0, 59.2)
- moved R6 26.9 mm to (84.4, 50.4)
- moved TP10 26.9 mm to (95.8, 39.6)
- moved TP5 26.9 mm to (83.3, 39.6)
- moved TP6 26.9 mm to (79.9, 39.6)
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Connections:
- U3 pad 10: /PWR_LED -> unconnected-(U3-P0.29-Pad10)
- U3 pad 11: /PAIR_LED -> unconnected-(U3-P0.02-Pad11)
- U3 pad 24: unconnected-(U3-P0.08-Pad24) -> /PAIR_LED
- U3 pad 26: unconnected-(U3-P1.09-Pad26) -> /MODE_SW
- U3 pad 4: /MODE_SW -> unconnected-(U3-P1.11-Pad4)
- U3 pad 46: unconnected-(U3-P0.22-Pad46) -> /PWR_LED
Routing:
- net +3V3: track 4.90 -> 157.5 mm, vias 0 -> 3
- net /PAIR_SW: track 0.00 -> 53.8 mm, vias 0 -> 2
- net /TIMING_PIN: track 0.00 -> 32.8 mm, vias 0 -> 1
- net /NRST: track 0.00 -> 30.4 mm, vias 0 -> 1
- net /P0.27: track 0.00 -> 28.8 mm
- net /MODE_SW: track 0.00 -> 27.1 mm, vias 0 -> 2
- net /DBG_TX: track 0.00 -> 25.6 mm
- net /AIN6: track 0.00 -> 25.1 mm
- net /SWDIO: track 0.00 -> 24.7 mm
- net /P0.26: track 0.00 -> 23.7 mm, vias 0 -> 2
- net VBUS: track 19.6 -> 40.8 mm
- net /SWO: track 0.00 -> 19.8 mm, vias 0 -> 1
- net /PAIR_LED: track 0.00 -> 19.6 mm, vias 0 -> 2
- net /AIN7: track 0.00 -> 18.7 mm
- net /DBG_RX: track 0.00 -> 18.7 mm
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- added copper zone on F.Cu, net +3V3
Other:
- board text added: "GPIO"
- board text added: "HID"
- board text added: "ON"
- board text added: "PAIR"
- board text added: "RST"
- board text added: "XINPUT"

Commit message: Clean up silkscreen labels on dongle PCB
Other:
- board text added: "DEBUG"
- board text added: "UART"
Changed lines of the file:
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@@
 		(tags "test point SMD pad rectangle square")
 		(property "Reference" "TP14"
-			(at 0 -1.448 270)
+			(at 0 -1.448 90)
 			(layer "F.SilkS")
 			(hide yes)
@@
 		)
 		(property "Value" "P0.04"
-			(at 0 1.55 270)
-			(layer "F.Fab")
+			(at 0 1.55 90)
+			(layer "F.SilkS")
 			(effects
 				(font
@@
 		)
 		(fp_text user "${REFERENCE}"
-			(at 0 -1.45 270)
+			(at 0 -1.45 90)
 			(layer "F.Fab")
 			(effects
@@
 		(tags "test point SMD pad rectangle square")
 		(property "Reference" "TP13"
-			(at 0 -1.448 270)
+			(at 0 -1.448 90)
 			(layer "F.SilkS")
 			(hide yes)
@@
 		)
 		(property "Value" "AIN7"
-			(at 0 1.55 270)
-			(layer "F.Fab")
+			(at 0 1.55 90)
+			(layer "F.SilkS")
 			(effects
 				(font
@@
 		)
 		(fp_text user "${REFERENCE}"
-			(at 0 -1.45 270)
+			(at 0 -1.45 90)
 			(layer "F.Fab")
 			(effects
@@
 		(tags "test point SMD pad rectangle square")
 		(property "Reference" "TP12"
-			(at 0 -1.448 270)
+			(at 0 -1.448 90)
 			(layer "F.SilkS")
 			(hide yes)
@@
 		)
 		(property "Value" "AIN6"
-			(at 0 1.55 270)
-			(layer "F.Fab")
+			(at 0 1.55 90)
+			(layer "F.SilkS")
 			(effects
 				(font
@@
 		)
 		(fp_text user "${REFERENCE}"
-			(at 0 -1.45 270)
+			(at 0 -1.45 90)
 			(layer "F.Fab")
 			(effects
@@
 		(tags "test point SMD pad rectangle square")
 		(property "Reference" "TP16"
-			(at 0 -1.448 270)
+			(at 0 -1.448 90)
 			(layer "F.SilkS")
 			(hide yes)
@@
 		)
 		(property "Value" "P0.26"
-			(at 0 1.55 270)
-			(layer "F.Fab")
+			(at 0 1.55 90)
+			(layer "F.SilkS")
 			(effects
 				(font
@@
 		)
 		(fp_text user "${REFERENCE}"
-			(at 0 -1.45 270)
+			(at 0 -1.45 90)
 			(layer "F.Fab")
 			(effects
@@
 		(tags "test point SMD pad rectangle square")
 		(property "Reference" "TP15"
-			(at 0 -1.448 270)
+			(at 0 -1.448 90)
 			(layer "F.SilkS")
 			(hide yes)
@@
 		)
 		(property "Value" "P0.06"
-			(at 0 1.55 270)
-			(layer "F.Fab")
+			(at 0 1.55 90)
+			(layer "F.SilkS")
 			(effects
 				(font
@@
 		)
 		(fp_text user "${REFERENCE}"
-			(at 0 -1.45 270)
+			(at 0 -1.45 90)
 			(layer "F.Fab")
 			(effects
@@
 		(tags "test point SMD pad rectangle square")
 		(property "Reference" "TP17"
-			(at 0 -1.448 270)
+			(at 0 -1.448 90)
 			(layer "F.SilkS")
 			(hide yes)
@@
 		)
 		(property "Value" "P0.27"
-			(at 0 1.55 270)
-			(layer "F.Fab")
+			(at 0 1.55 90)
+			(layer "F.SilkS")
 			(effects
 				(font
@@
 		)
 		(fp_text user "${REFERENCE}"
-			(at 0 -1.45 270)
+			(at 0 -1.45 90)
 			(layer "F.Fab")
 			(effects
@@
 		(layer "Edge.Cuts")
 	)
+	(gr_text "UART"
+		(at 76.35 70.35 270)
+		(layer "F.SilkS")
+		(effects
+			(font
+				(size 1 1)
+				(thickness 0.15)
+			)
+		)
+	)
+	(gr_text "DEBUG"
+		(at 76.35 77.875 270)
+		(layer "F.SilkS")
+		(effects
+			(font
+				(size 1 1)
+				(thickness 0.15)
+			)
+		)
+	)
 	(gr_text "PAIR"

Commit message: Add JP1 silkscreen warning for dongle PCB
Other:
- board text added: "IO"
- board text added: "ONLY BRIDGE ONE SIDE"
- board text removed: "GPIO"
Changed lines of the file:
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@@
+		)
+	)
+	(gr_text "ONLY BRIDGE\nONE SIDE"
+		(at 94.675 68.375 270)
+		(layer "F.SilkS")
+		(effects
+			(font
+				(size 1 1)
+				(thickness 0.15)
+			)
 		)
 	)
@@
 		)
 	)
-	(gr_text "GPIO"
-		(at 89.5 65.325 0)
+	(gr_text "ON"
+		(at 90.225 73.425 0)
 		(layer "F.SilkS")
 		(effects
@@
 		)
 	)
-	(gr_text "ON"
-		(at 90.375 73.325 0)
+	(gr_text "IO"
+		(at 90.85 65.25 0)
 		(layer "F.SilkS")
 		(effects

Commit message: Dongle PCB Rev1.1 ready for fab
Other:
- board text added: "XBX-NRF Gamepad Dongle Rev ${REV} https://github.com/zuidec/xbx-nrf"
Changed lines of the file:
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@@
 		(title "XBX-NRF Gamepad Dongle PCB Layout")
 		(date "2026-10-02")
-		(rev "1")
+		(rev "${REV}")
 	)
 	(layers
@@
 		)
 		(pad_to_mask_clearance 0)
-		(solder_mask_min_width 0.1)
 		(allow_soldermask_bridges_in_footprints no)
 		(tenting
@@
 		)
 	)
+	(property "REV" "1.1")
 	(footprint "xbx-nrf-lib:TestPoint_Pad_1.0x1.0mm-NoSilkscreen"
 		(layer "F.Cu")
@@
 		)
 	)
+	(gr_text "XBX-NRF Gamepad Dongle\nRev ${REV}\nhttps://github.com/zuidec/xbx-nrf"
+		(at 102.4 42.55 90)
+		(layer "B.SilkS")
+		(effects
+			(font
+				(size 1.5 1.5)
+				(thickness 0.3)
+				(bold yes)
+			)
+			(justify left bottom mirror)
+		)
+	)
 	(gr_text "ANTENNA ZONE"
 		(at 126.831804 66.472865 90)
@@
 			(layer "Dwgs.User")
 			(effects
-				(font
-					(size 1 1)
-					(thickness 0.15)
-				)
-			)
-		)
-	)
-	(dimension
-		(type orthogonal)
-		(layer "Dwgs.User")
-		(pts
-			(xy 79.88 100.3) (xy 80.155 95.3)
-		)
-		(height -0.155)
-		(orientation 1)
-		(format
-			(prefix "")
-			(suffix "")
-			(units 3)
-			(units_format 0)
-			(precision 4)
-			(suppress_zeroes yes)
-		)
-		(style
-			(thickness 0.1)
-			(arrow_length 1.27)
-			(text_position_mode 0)
-			(arrow_direction outward)
-			(extension_height 0.58642)
-			(extension_offset 0.5)
-			(keep_text_aligned yes)
-		)
-		(gr_text "5"
-			(at 78.575 97.8 90)
-			(layer "Dwgs.User")
-			(effects

Commit message: Fix: debug TX/RX pins are reversed
Connections:
- J3 pad 1: /DBG_RX -> /DBG_TX
- J3 pad 3: /DBG_TX -> /DBG_RX
- U3 pad 43: /DBG_TX -> /DBG_RX
- U3 pad 44: /DBG_RX -> /DBG_TX
Routing:
- net /DBG_TX: track 25.6 -> 18.7 mm
- net /DBG_RX: track 18.7 -> 25.6 mm
Changed lines of the file:
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@@
 			(size 0.6 0.4)
 			(layers "F.Cu" "F.Mask" "F.Paste")
-			(net "/DBG_TX")
+			(net "/DBG_RX")
 			(pinfunction "P0.21_43")
 			(pintype "bidirectional")
@@
 			(size 0.6 0.4)
 			(layers "F.Cu" "F.Mask" "F.Paste")
-			(net "/DBG_RX")
+			(net "/DBG_TX")
 			(pinfunction "P0.20_44")
 			(pintype "bidirectional")
@@
 			(layers "F.Cu" "F.Mask" "F.Paste")
 			(roundrect_rratio 0.25)
-			(net "/DBG_RX")
+			(net "/DBG_TX")
 			(pinfunction "Pin_1_1")
 			(pintype "passive")
@@
 			(layers "F.Cu" "F.Mask" "F.Paste")
 			(roundrect_rratio 0.25)
-			(net "/DBG_TX")
+			(net "/DBG_RX")
 			(pinfunction "Pin_3_3")
 			(pintype "passive")
@@
 	)
 	(segment
-		(start 98.106804 65.272865)
-		(end 97.481804 64.647865)
+		(start 90.456804 65.397865)
+		(end 90.656804 65.197865)
 		(width 0.15)
 		(layer "F.Cu")
@@
 	)
 	(segment
-		(start 97.481804 64.647865)
-		(end 87.981804 64.647865)
+		(start 95.481804 65.672865)
+		(end 97.406804 65.672865)
 		(width 0.15)
 		(layer "F.Cu")
@@
 	)
 	(segment
-		(start 81.256805 71.572865)
-		(end 82.031804 71.572865)
+		(start 82.031804 69.572865)
+		(end 82.031804 67.322865)
 		(width 0.15)
 		(layer "F.Cu")
@@
 	)
 	(segment
-		(start 87.981804 64.647865)
-		(end 85.956804 66.672865)
+		(start 85.956804 67.222865)
+		(end 87.781804 65.397865)
 		(width 0.15)
 		(layer "F.Cu")
@@
 	)
 	(segment
-		(start 79.756804 67.218196)
-		(end 79.756804 70.072864)
+		(start 95.006804 65.197865)
+		(end 95.481804 65.672865)
 		(width 0.15)
 		(layer "F.Cu")
@@
 	)
 	(segment
-		(start 79.756804 70.072864)
-		(end 81.256805 71.572865)
+		(start 90.656804 65.197865)
+		(end 95.006804 65.197865)
 		(width 0.15)
 		(layer "F.Cu")
@@
 	)
 	(segment
-		(start 85.956804 66.672865)
-		(end 80.302135 66.672865)
+		(start 82.031804 67.322865)
+		(end 82.131804 67.222865)
 		(width 0.15)
 		(layer "F.Cu")
@@
 	)
 	(segment
-		(start 98.306804 65.272865)
-		(end 98.106804 65.272865)
+		(start 87.781804 65.397865)
+		(end 90.456804 65.397865)
 		(width 0.15)
 		(layer "F.Cu")
@@
 	)
 	(segment
-		(start 80.302135 66.672865)
-		(end 79.756804 67.218196)
+		(start 82.131804 67.222865)
+		(end 85.956804 67.222865)
 		(width 0.15)
 		(layer "F.Cu")
@@
 	)
 	(segment
-		(start 90.456804 65.397865)
-		(end 90.656804 65.197865)
+		(start 98.106804 65.272865)
+		(end 97.481804 64.647865)
 		(width 0.15)
 		(layer "F.Cu")
@@
 	)
 	(segment
-		(start 95.481804 65.672865)
-		(end 97.406804 65.672865)
+		(start 97.481804 64.647865)
+		(end 87.981804 64.647865)
 		(width 0.15)
 		(layer "F.Cu")
@@
 	)
 	(segment
-		(start 82.031804 69.572865)
-		(end 82.031804 67.322865)
+		(start 81.256805 71.572865)
+		(end 82.031804 71.572865)
 		(width 0.15)
 		(layer "F.Cu")
@@
 	)
 	(segment
-		(start 85.956804 67.222865)
-		(end 87.781804 65.397865)
+		(start 87.981804 64.647865)
+		(end 85.956804 66.672865)
 		(width 0.15)
 		(layer "F.Cu")
@@
 	)
 	(segment
-		(start 95.006804 65.197865)
-		(end 95.481804 65.672865)
+		(start 79.756804 67.218196)
+		(end 79.756804 70.072864)
 		(width 0.15)
 		(layer "F.Cu")
@@
 	)
 	(segment
-		(start 90.656804 65.197865)
-		(end 95.006804 65.197865)
+		(start 79.756804 70.072864)
+		(end 81.256805 71.572865)
 		(width 0.15)
 		(layer "F.Cu")
@@
 	)
 	(segment
-		(start 82.031804 67.322865)
-		(end 82.131804 67.222865)
+		(start 85.956804 66.672865)
+		(end 80.302135 66.672865)
 		(width 0.15)
 		(layer "F.Cu")
@@
 	)
 	(segment
-		(start 87.781804 65.397865)
-		(end 90.456804 65.397865)
+		(start 98.306804 65.272865)
+		(end 98.106804 65.272865)
 		(width 0.15)
 		(layer "F.Cu")
@@
 	)
 	(segment
-		(start 82.131804 67.222865)
-		(end 85.956804 67.222865)
+		(start 80.302135 66.672865)
+		(end 79.756804 67.218196)
 		(width 0.15)
 		(layer "F.Cu")
