File: pcb/xbx-nrf-dongle/xbx-nrf-dongle.kicad_sch (KiCad schematic)
At the start: 57 parts, among them J1 SWD, J2 UART, J3 16P-USBC-RECEPTACLE, SW1 SW_Push, SW2 SW_Push, SW3 SW_SPDT, U1 LDS3985M33R_SOT23, U2 USBLC6-2SC6, U3 MDBT50Q-U1MV2, Y1 32.768kHz

Commit message: Rev1 positioning complete, pre-routing commit
Parts:
- J1, J2: symbol Connector:Conn_01x03_Socket -> Connector_Generic_MountingPin:Conn_01x03_MountingPin
- TP1, TP2, TP3, TP4: footprint TestPoint:TestPoint_Pad_2.0x2.0mm -> TestPoint:TestPoint_Pad_1.5x1.5mm
- TP10, TP11, TP12, TP13, TP14, TP15, TP16, TP17, TP5, TP6, TP7, TP8, TP9: footprint TestPoint:TestPoint_Pad_2.0x2.0mm -> TestPoint:TestPoint_Pad_1.0x1.0mm
Connections:
- net GND: now also J1.MP (MountPin), J2.MP (MountPin)
- net D+_EXT renamed EXT_D+
- net D-_EXT renamed EXT_D-
Changed lines of the file:
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@@
 	)
 	(junction
+		(at 245.11 45.72)
+		(diameter 0)
+		(color 0 0 0 0)
+	)
+	(junction
 		(at 26.67 78.74)
 		(diameter 0)
@@
 	)
 	(junction
+		(at 245.11 27.94)
+		(diameter 0)
+		(color 0 0 0 0)
+	)
+	(junction
 		(at 140.97 24.13)
 		(diameter 0)
@@
 	(wire
 		(pts
-			(xy 232.41 43.18) (xy 240.03 43.18)
+			(xy 232.41 48.26) (xy 240.03 48.26)
 		)
 		(stroke
@@
 	(wire
 		(pts
+			(xy 245.11 17.78) (xy 245.11 27.94)
+		)
+		(stroke
+			(width 0)
+			(type default)
+		)
+	)
+	(wire
+		(pts
 			(xy 113.03 24.13) (xy 115.57 24.13)
 		)
@@
 	(wire
 		(pts
+			(xy 227.33 35.56) (xy 245.11 35.56)
+		)
+		(stroke
+			(width 0)
+			(type default)
+		)
+	)
+	(wire
+		(pts
 			(xy 17.78 78.74) (xy 17.78 73.66)
 		)
@@
 	(wire
 		(pts
+			(xy 227.33 17.78) (xy 245.11 17.78)
+		)
+		(stroke
+			(width 0)
+			(type default)
+		)
+	)
+	(wire
+		(pts
 			(xy 86.36 33.02) (xy 73.66 33.02)
 		)
@@
 	(wire
 		(pts
-			(xy 232.41 38.1) (xy 240.03 38.1)
+			(xy 232.41 43.18) (xy 240.03 43.18)
 		)
 		(stroke
@@
 	(wire
 		(pts
+			(xy 227.33 38.1) (xy 227.33 35.56)
+		)
+		(stroke
+			(width 0)
+			(type default)
+		)
+	)
+	(wire
+		(pts
 			(xy 86.36 138.43) (xy 91.44 138.43)
 		)
@@
 	(wire
 		(pts
-			(xy 232.41 40.64) (xy 245.11 40.64)
+			(xy 232.41 45.72) (xy 245.11 45.72)
 		)
 		(stroke
@@
 	(wire
 		(pts
+			(xy 227.33 20.32) (xy 227.33 17.78)
+		)
+		(stroke
+			(width 0)
+			(type default)
+		)
+	)
+	(wire
+		(pts
 			(xy 17.78 87.63) (xy 26.67 87.63)
 		)
@@
 	(wire
 		(pts
+			(xy 245.11 35.56) (xy 245.11 45.72)
+		)
+		(stroke
+			(width 0)
+			(type default)
+		)
+	)
+	(wire
+		(pts
 			(xy 151.13 104.14) (xy 154.94 104.14)
 		)
@@
 		)
 	)
-	(label "D-_EXT"
+	(label "EXT_D-"
 		(at 69.85 40.64 180)
 		(effects
@@
 		)
 	)
-	(label "D+_EXT"
+	(label "EXT_D+"
 		(at 69.85 43.18 180)
 		(effects
@@
 		)
 	)
-	(label "D-_EXT"
+	(label "EXT_D-"
 		(at 16.51 43.18 0)
 		(effects
@@
 		)
 	)
-	(label "D+_EXT"
+	(label "EXT_D+"
 		(at 16.51 40.64 0)
 		(effects
@@
 	)
 	(label "DBG_RX"
-		(at 240.03 43.18 180)
+		(at 240.03 48.26 180)
 		(effects
 			(font
@@
 	)
 	(label "DBG_TX"
-		(at 240.03 38.1 180)
+		(at 240.03 43.18 180)
 		(effects
 			(font
@@
 		)
 	)
-	(label "D+_EXT"
+	(label "EXT_D+"
 		(at 72.39 43.18 0)
 		(effects
@@
 		)
 	)
-	(label "D-_EXT"
+	(label "EXT_D-"
 		(at 72.39 45.72 0)
 		(effects
@@
 			)
 		)
-		(property "Footprint" "TestPoint:TestPoint_Pad_2.0x2.0mm"
+		(property "Footprint" "TestPoint:TestPoint_Pad_1.0x1.0mm"
 			(at 22.86 73.66 0)
 			(hide yes)
@@
 			)
 		)
-		(property "Footprint" "TestPoint:TestPoint_Pad_2.0x2.0mm"
+		(property "Footprint" "TestPoint:TestPoint_Pad_1.0x1.0mm"
 			(at 44.45 115.57 0)
 			(hide yes)
@@
 			)
 		)
-		(property "Footprint" "TestPoint:TestPoint_Pad_2.0x2.0mm"
+		(property "Footprint" "TestPoint:TestPoint_Pad_1.0x1.0mm"
 			(at 40.64 82.55 0)
 			(hide yes)
@@
 			)
 		)
-		(property "Footprint" "TestPoint:TestPoint_Pad_2.0x2.0mm"
+		(property "Footprint" "TestPoint:TestPoint_Pad_1.0x1.0mm"
 			(at 31.75 82.55 0)
 			(hide yes)
@@
 			)
 		)
-		(property "Footprint" "TestPoint:TestPoint_Pad_2.0x2.0mm"
+		(property "Footprint" "TestPoint:TestPoint_Pad_1.0x1.0mm"
 			(at 22.86 82.55 0)
 			(hide yes)
@@
 		(in_pos_files yes)
 		(dnp no)
-		(fields_autoplaced yes)
 		(property "Reference" "#PWR07"
 			(at 245.11 34.29 0)
@@
 		)
 		(property "Value" "GND"
-			(at 245.11 33.02 0)
+			(at 245.11 32.512 0)
 			(show_name no)
 			(do_not_autoplace no)
@@
 			)
 		)
-		(property "Footprint" "TestPoint:TestPoint_Pad_2.0x2.0mm"
+		(property "Footprint" "TestPoint:TestPoint_Pad_1.0x1.0mm"
 			(at 33.02 115.57 0)
 			(hide yes)
@@
 			)
 		)
-		(property "Footprint" "TestPoint:TestPoint_Pad_2.0x2.0mm"
+		(property "Footprint" "TestPoint:TestPoint_Pad_1.5x1.5mm"
 			(at 278.13 39.37 0)
 			(hide yes)
@@
 			)
 		)
-		(property "Footprint" "TestPoint:TestPoint_Pad_2.0x2.0mm"
+		(property "Footprint" "TestPoint:TestPoint_Pad_1.0x1.0mm"
 			(at 33.02 104.14 0)
 			(hide yes)
@@
 			)
 		)
-		(property "Footprint" "TestPoint:TestPoint_Pad_2.0x2.0mm"
+		(property "Footprint" "TestPoint:TestPoint_Pad_1.0x1.0mm"
 			(at 44.45 104.14 0)
 			(hide yes)
@@
 			)
 		)
-		(property "Footprint" "TestPoint:TestPoint_Pad_2.0x2.0mm"
+		(property "Footprint" "TestPoint:TestPoint_Pad_1.0x1.0mm"
 			(at 31.75 73.66 0)
 			(hide yes)
@@
 			)
 		)
-		(property "Footprint" "TestPoint:TestPoint_Pad_2.0x2.0mm"
+		(property "Footprint" "TestPoint:TestPoint_Pad_1.5x1.5mm"
 			(at 259.08 39.37 0)
 			(hide yes)
@@
 	)
 	(symbol
-		(lib_id "Connector:Conn_01x03_Socket")
+		(lib_id "Connector_Generic_MountingPin:Conn_01x03_MountingPin")
 		(at 227.33 27.94 180)
 		(unit 1)
@@
 			)
 		)
-		(property "Description" "Generic connector, single row, 01x03, script generated"
+		(property "Description" "Generic connectable mounting pin connector, single row, 01x03, script generated (kicad-library-utils/schlib/autogen/connector/)"
 			(at 227.33 27.94 0)
 			(hide yes)
@@
 		(pin "1"
 		)
+		(pin "MP"
+		)
 		(instances
 			(project "xbx-nrf-dongle"
@@
 			)
 		)
-		(property "Footprint" "TestPoint:TestPoint_Pad_2.0x2.0mm"
+		(property "Footprint" "TestPoint:TestPoint_Pad_1.0x1.0mm"
 			(at 22.86 90.17 0)
 			(hide yes)
@@
 	)
 	(symbol
-		(lib_id "Connector:Conn_01x03_Socket")
-		(at 227.33 40.64 180)
+		(lib_id "Connector_Generic_MountingPin:Conn_01x03_MountingPin")
+		(at 227.33 45.72 180)
 		(unit 1)
 		(body_style 1)
@@
 		(dnp no)
 		(property "Reference" "J2"
-			(at 230.632 32.512 0)
+			(at 230.632 37.592 0)
 			(show_name no)
 			(do_not_autoplace no)
@@
 		)
 		(property "Value" "UART"
-			(at 230.632 35.052 0)
+			(at 230.632 40.132 0)
 			(show_name no)
 			(do_not_autoplace no)
@@
 		)
 		(property "Footprint" "Connector_JST:JST_SH_SM03B-SRSS-TB_1x03-1MP_P1.00mm_Horizontal"
-			(at 227.33 40.64 0)
+			(at 227.33 45.72 0)
 			(hide yes)
 			(show_name no)
@@
 		)
 		(property "Datasheet" ""
-			(at 227.33 40.64 0)
+			(at 227.33 45.72 0)
 			(hide yes)
 			(show_name no)
@@
 			)
 		)
-		(property "Description" "Generic connector, single row, 01x03, script generated"
-			(at 227.33 40.64 0)
+		(property "Description" "Generic connectable mounting pin connector, single row, 01x03, script generated (kicad-library-utils/schlib/autogen/connector/)"
+			(at 227.33 45.72 0)
 			(hide yes)
 			(show_name no)
@@
 		(pin "1"
 		)
+		(pin "MP"
+		)
 		(instances
 			(project "xbx-nrf-dongle"
@@
 			)
 		)
-		(property "Footprint" "TestPoint:TestPoint_Pad_2.0x2.0mm"
+		(property "Footprint" "TestPoint:TestPoint_Pad_1.5x1.5mm"
 			(at 269.24 39.37 0)
 			(hide yes)
@@
 			)
 		)
-		(property "Footprint" "TestPoint:TestPoint_Pad_2.0x2.0mm"
+		(property "Footprint" "TestPoint:TestPoint_Pad_1.0x1.0mm"
 			(at 40.64 73.66 0)
 			(hide yes)
@@
 			)
 		)
-		(property "Footprint" "TestPoint:TestPoint_Pad_2.0x2.0mm"
+		(property "Footprint" "TestPoint:TestPoint_Pad_1.0x1.0mm"
 			(at 21.59 104.14 0)
 			(hide yes)
@@
 			)
 		)
-		(property "Footprint" "TestPoint:TestPoint_Pad_2.0x2.0mm"
+		(property "Footprint" "TestPoint:TestPoint_Pad_1.5x1.5mm"
 			(at 256.54 16.51 0)
 			(hide yes)
@@
 			)
 		)
-		(property "Footprint" "TestPoint:TestPoint_Pad_2.0x2.0mm"
+		(property "Footprint" "TestPoint:TestPoint_Pad_1.0x1.0mm"
 			(at 21.59 115.57 0)
 			(hide yes)
@@
 	(symbol
 		(lib_id "power:GND")
-		(at 245.11 40.64 0)
+		(at 245.11 45.72 0)
 		(unit 1)
 		(body_style 1)
@@
 		(fields_autoplaced yes)
 		(property "Reference" "#PWR014"
-			(at 245.11 46.99 0)
+			(at 245.11 52.07 0)
 			(hide yes)
 			(show_name no)
@@
 		)
 		(property "Value" "GND"
-			(at 245.11 45.72 0)
+			(at 245.11 50.8 0)
 			(show_name no)
 			(do_not_autoplace no)
@@
 		)
 		(property "Footprint" ""
-			(at 245.11 40.64 0)
+			(at 245.11 45.72 0)
 			(hide yes)
 			(show_name no)
@@
 		)
 		(property "Datasheet" ""
-			(at 245.11 40.64 0)
+			(at 245.11 45.72 0)
 			(hide yes)
 			(show_name no)
@@
 		)
 		(property "Description" "Power symbol creates a global label with name \"GND\" , ground"
-			(at 245.11 40.64 0)
+			(at 245.11 45.72 0)
 			(hide yes)
 			(show_name no)

Commit message: Change board shape, reposition components. Pre-routing commit
Parts:
- removed C4: 1uF, Capacitor_SMD:C_0603_1608Metric_Pad1.08x0.95mm_HandSolder, symbol Device:C_Small
- removed H2: MountingHole, MountingHole:MountingHole_2.2mm_M2, symbol Mechanical:MountingHole
- removed R3: 10k, Resistor_SMD:R_0603_1608Metric_Pad0.98x0.95mm_HandSolder, symbol Device:R_Small
- renumbered C5 to C4, C6 to C5, C7 to C6, C8 to C7, H3 to H2, J3 to J2, J2 to J3, R11 to R10, R12 to R11, R4 to R3, R5 to R4, R6 to R5, R7 to R6, R8 to R7, R9 to R8, R10 to R9
Connections:
- net +3V3: no longer R1.1
- net D+: now also R4.2; no longer R3.1
- net D-: now also R3.1; no longer R4.2
- net EXT_D+: now also U2.3 (I/O2); no longer U2.1 (I/O1)
- net EXT_D-: now also U2.1 (I/O1); no longer U2.3 (I/O2)
- net GND: now also R1.1
- net XL1: now reaches C6.2, U3.17 (P0.00), Y1.1
- net XL2: now reaches C7.1, U3.18 (P0.01), Y1.2
- no-connect marks 30 -> 31
Other:
- moved on the sheet: H2

Commit message: Dongle PCB Rev1 complete
Parts:
- J2: footprint usbc-16p-receptacle-amphenol:USB_C_Receptacle_16P_Amphenol_10155435-00011LF -> xbx-nrf-lib:USB_C_Receptacle_16P_Amphenol_10155435-00011LF
- JP1: footprint Jumper:SolderJumper-3_P2.0mm_Open_TrianglePad1.0x1.5mm_NumberLabels -> xbx-nrf-lib:SolderJumper-3_P2.0mm_Open_TrianglePad1.0x1.5mm_NumberLabels; private KLC_S3.3 -> (none)
- R1: value 10k -> 1k
- TP1, TP2, TP3, TP4: footprint TestPoint:TestPoint_Pad_1.5x1.5mm -> xbx-nrf-lib:TestPoint_Pad_1.5x1.5mm-NoSilkscreen
- TP10, TP11, TP12, TP13, TP14, TP15, TP16, TP17, TP5, TP6, TP7, TP8, TP9: footprint TestPoint:TestPoint_Pad_1.0x1.0mm -> xbx-nrf-lib:TestPoint_Pad_1.0x1.0mm-NoSilkscreen
- U3: footprint RF_Module:Raytac_MDBT50Q -> xbx-nrf-lib:Raytac_MDBT50Q
- Y1: footprint Crystal:Crystal_SMD_3215-2Pin_3.2x1.5mm -> xbx-nrf-lib:Crystal_SMD_3215-2Pin_3.2x1.5mm
Connections:
- net MODE_SW: now also U3.26 (P1.09); no longer U3.4 (P1.11)
- net PAIR_LED: now also U3.24 (P0.08); no longer U3.11 (P0.02)
- net PWR_LED: now also U3.46 (P0.22); no longer U3.10 (P0.29)
Changed lines of the file:
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@@
 	)
 	(no_connect
+		(at 91.44 115.57)
+	)
+	(no_connect
 		(at 91.44 128.27)
 	)
@@
 	)
 	(no_connect
-		(at 132.08 143.51)
-	)
-	(no_connect
 		(at 24.13 45.72)
 	)
@@
 	)
 	(no_connect
+		(at 91.44 102.87)
+	)
+	(no_connect
 		(at 132.08 115.57)
 	)
@@
 	)
 	(no_connect
-		(at 207.01 34.29)
+		(at 91.44 166.37)
 	)
 	(no_connect
-		(at 132.08 110.49)
+		(at 207.01 34.29)
 	)
 	(no_connect
@@
 	)
 	(no_connect
-		(at 132.08 168.91)
-	)
-	(no_connect
 		(at 132.08 163.83)
 	)
@@
 	(wire
 		(pts
-			(xy 132.08 100.33) (xy 149.86 100.33)
+			(xy 132.08 110.49) (xy 142.24 110.49)
 		)
 		(stroke
@@
 	(wire
 		(pts
-			(xy 81.28 115.57) (xy 91.44 115.57)
+			(xy 132.08 100.33) (xy 149.86 100.33)
 		)
 		(stroke
@@
 	(wire
 		(pts
+			(xy 132.08 168.91) (xy 143.51 168.91)
+		)
+		(stroke
+			(width 0)
+			(type default)
+		)
+	)
+	(wire
+		(pts
 			(xy 265.43 64.77) (xy 281.94 64.77)
 		)
@@
 	(wire
 		(pts
-			(xy 80.01 166.37) (xy 91.44 166.37)
-		)
-		(stroke
-			(width 0)
-			(type default)
-		)
-	)
-	(wire
-		(pts
 			(xy 140.97 24.13) (xy 148.59 24.13)
 		)
@@
 	(wire
 		(pts
-			(xy 80.01 102.87) (xy 91.44 102.87)
-		)
-		(stroke
-			(width 0)
-			(type default)
-		)
-	)
-	(wire
-		(pts
 			(xy 250.19 82.55) (xy 265.43 82.55)
 		)
@@
 	(wire
 		(pts
+			(xy 132.08 143.51) (xy 142.24 143.51)
+		)
+		(stroke
+			(width 0)
+			(type default)
+		)
+	)
+	(wire
+		(pts
 			(xy 35.56 78.74) (xy 26.67 78.74)
 		)
@@
 		)
 	)
+	(label "MODE_SW"
+		(at 143.51 168.91 180)
+		(effects
+			(font
+				(size 1.27 1.27)
+			)
+			(justify right bottom)
+		)
+	)
 	(label "SWO"
 		(at 264.16 48.26 90)
@@
 		)
 	)
+	(label "PWR_LED"
+		(at 142.24 143.51 180)
+		(effects
+			(font
+				(size 1.27 1.27)
+			)
+			(justify right bottom)
+		)
+	)
 	(label "D+"
 		(at 86.36 138.43 0)
@@
 		)
 	)
-	(label "PAIR_LED"
-		(at 80.01 102.87 0)
-		(effects
-			(font
-				(size 1.27 1.27)
-			)
-			(justify left bottom)
-		)
-	)
 	(label "MODE_SW"
 		(at 191.77 38.1 90)
@@
 		)
 	)
+	(label "PAIR_LED"
+		(at 142.24 110.49 180)
+		(effects
+			(font
+				(size 1.27 1.27)
+			)
+			(justify right bottom)
+		)
+	)
 	(label "SWO"
 		(at 138.43 161.29 180)
@@
 		)
 	)
-	(label "PWR_LED"
-		(at 81.28 115.57 0)
-		(effects
-			(font
-				(size 1.27 1.27)
-			)
-			(justify left bottom)
-		)
-	)
 	(label "P0.26"
 		(at 27.94 123.19 90)
@@
 		)
 	)
-	(label "MODE_SW"
-		(at 80.01 166.37 0)
-		(effects
-			(font
-				(size 1.27 1.27)
-			)
-			(justify left bottom)
-		)
-	)
 	(label "P3_LED"
 		(at 260.35 97.79 180)
@@
 			)
 		)
-		(property "Footprint" "TestPoint:TestPoint_Pad_1.0x1.0mm"
+		(property "Footprint" "xbx-nrf-lib:TestPoint_Pad_1.0x1.0mm-NoSilkscreen"
 			(at 22.86 73.66 0)
 			(hide yes)
@@
 			)
 		)
-		(property "Value" "10k"
+		(property "Value" "1k"
 			(at 209.55 26.6699 0)
 			(show_name no)
@@
 			)
 		)
-		(property "Footprint" "TestPoint:TestPoint_Pad_1.0x1.0mm"
+		(property "Footprint" "xbx-nrf-lib:TestPoint_Pad_1.0x1.0mm-NoSilkscreen"
 			(at 44.45 115.57 0)
 			(hide yes)
@@
 			)
 		)
-		(property "Footprint" "Crystal:Crystal_SMD_3215-2Pin_3.2x1.5mm"
+		(property "Footprint" "xbx-nrf-lib:Crystal_SMD_3215-2Pin_3.2x1.5mm"
 			(at 154.94 101.6 0)
 			(hide yes)
@@
 			)
 		)
-		(property "Footprint" "TestPoint:TestPoint_Pad_1.0x1.0mm"
+		(property "Footprint" "xbx-nrf-lib:TestPoint_Pad_1.0x1.0mm-NoSilkscreen"
 			(at 40.64 82.55 0)
 			(hide yes)
@@
 			)
 		)
-		(property "Footprint" "TestPoint:TestPoint_Pad_1.0x1.0mm"
+		(property "Footprint" "xbx-nrf-lib:TestPoint_Pad_1.0x1.0mm-NoSilkscreen"
 			(at 31.75 82.55 0)
 			(hide yes)
@@
 			)
 		)
-		(property "Footprint" "TestPoint:TestPoint_Pad_1.0x1.0mm"
+		(property "Footprint" "xbx-nrf-lib:TestPoint_Pad_1.0x1.0mm-NoSilkscreen"
 			(at 22.86 82.55 0)
 			(hide yes)
@@
 			)
 		)
-		(property "Footprint" "Jumper:SolderJumper-3_P2.0mm_Open_TrianglePad1.0x1.5mm_NumberLabels"
+		(property "Footprint" "xbx-nrf-lib:SolderJumper-3_P2.0mm_Open_TrianglePad1.0x1.5mm_NumberLabels"
 			(at 252.73 111.76 0)
 			(hide yes)
@@
 			)
 		)
-		(property private "KLC_S5.1" "This is a generic symbol, it has fp-filter, but no default footprint"
-			(at 270.51 111.76 0)
-			(hide yes)
-			(show_name yes)
-			(do_not_autoplace no)
-			(effects
-				(font
-					(size 1.27 1.27)
-				)
-			)
-		)
-		(property private "KLC_S3.3" "Graphical-Symbol: thickness is 6mm, fill is background"
-			(at 273.05 111.76 0)
-			(hide yes)
-			(show_name yes)
-			(do_not_autoplace no)
-			(effects
-				(font
-					(size 1.27 1.27)
-				)
-			)
-		)
 		(pin "2"
 		)
@@
 			)
 		)
-		(property "Footprint" "TestPoint:TestPoint_Pad_1.0x1.0mm"
+		(property "Footprint" "xbx-nrf-lib:TestPoint_Pad_1.0x1.0mm-NoSilkscreen"
 			(at 33.02 115.57 0)
 			(hide yes)
@@
 			)
 		)
-		(property "Footprint" "TestPoint:TestPoint_Pad_1.5x1.5mm"
+		(property "Footprint" "xbx-nrf-lib:TestPoint_Pad_1.5x1.5mm-NoSilkscreen"
 			(at 278.13 39.37 0)
 			(hide yes)
@@
 			)
 		)
-		(property "Footprint" "TestPoint:TestPoint_Pad_1.0x1.0mm"
+		(property "Footprint" "xbx-nrf-lib:TestPoint_Pad_1.0x1.0mm-NoSilkscreen"
 			(at 33.02 104.14 0)
 			(hide yes)
@@
 			)
 		)
-		(property "Footprint" "TestPoint:TestPoint_Pad_1.0x1.0mm"
+		(property "Footprint" "xbx-nrf-lib:TestPoint_Pad_1.0x1.0mm-NoSilkscreen"
 			(at 44.45 104.14 0)
 			(hide yes)
@@
 			)
 		)
-		(property "Footprint" "TestPoint:TestPoint_Pad_1.0x1.0mm"
+		(property "Footprint" "xbx-nrf-lib:TestPoint_Pad_1.0x1.0mm-NoSilkscreen"
 			(at 31.75 73.66 0)
 			(hide yes)
@@
 			)
 		)
-		(property "Footprint" "TestPoint:TestPoint_Pad_1.5x1.5mm"
+		(property "Footprint" "xbx-nrf-lib:TestPoint_Pad_1.5x1.5mm-NoSilkscreen"
 			(at 259.08 39.37 0)
 			(hide yes)
@@
 			)
 		)
-		(property "Footprint" "TestPoint:TestPoint_Pad_1.0x1.0mm"
+		(property "Footprint" "xbx-nrf-lib:TestPoint_Pad_1.0x1.0mm-NoSilkscreen"
 			(at 22.86 90.17 0)
 			(hide yes)
@@
 			)
 		)
-		(property "Footprint" "usbc-16p-receptacle-amphenol:USB_C_Receptacle_16P_Amphenol_10155435-00011LF"
+		(property "Footprint" "xbx-nrf-lib:USB_C_Receptacle_16P_Amphenol_10155435-00011LF"
 			(at 41.91 43.18 0)
 			(hide yes)
@@
 			)
 		)
-		(property "Footprint" "TestPoint:TestPoint_Pad_1.5x1.5mm"
+		(property "Footprint" "xbx-nrf-lib:TestPoint_Pad_1.5x1.5mm-NoSilkscreen"
 			(at 269.24 39.37 0)
 			(hide yes)
@@
 			)
 		)
-		(property "Footprint" "TestPoint:TestPoint_Pad_1.0x1.0mm"
+		(property "Footprint" "xbx-nrf-lib:TestPoint_Pad_1.0x1.0mm-NoSilkscreen"
 			(at 40.64 73.66 0)
 			(hide yes)
@@
 			)
 		)
-		(property "Footprint" "TestPoint:TestPoint_Pad_1.0x1.0mm"
+		(property "Footprint" "xbx-nrf-lib:TestPoint_Pad_1.0x1.0mm-NoSilkscreen"
 			(at 21.59 104.14 0)
 			(hide yes)
@@
 			)
 		)
-		(property "Footprint" "TestPoint:TestPoint_Pad_1.5x1.5mm"
+		(property "Footprint" "xbx-nrf-lib:TestPoint_Pad_1.5x1.5mm-NoSilkscreen"
 			(at 256.54 16.51 0)
 			(hide yes)
@@
 			)
 		)
-		(property "Footprint" "TestPoint:TestPoint_Pad_1.0x1.0mm"
+		(property "Footprint" "xbx-nrf-lib:TestPoint_Pad_1.0x1.0mm-NoSilkscreen"
 			(at 21.59 115.57 0)
 			(hide yes)
@@
 			)
 		)
-		(property "Footprint" "RF_Module:Raytac_MDBT50Q"
+		(property "Footprint" "xbx-nrf-lib:Raytac_MDBT50Q"
 			(at 111.76 140.97 0)
 			(hide yes)

Commit message: Add title and date to dongle PCB sheets
Other:
- title: XBX-NRF Gamepad Dongle -> XBX-NRF Gamepad Dongle Schematic
Changed lines of the file:
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@@
 	(paper "A4")
 	(title_block
-		(title "XBX-NRF Gamepad Dongle")
+		(title "XBX-NRF Gamepad Dongle Schematic")
+		(date "2026-10-02")
 		(rev "1")
 	)

Commit message: Fix: debug TX/RX pins are reversed
Connections:
- net DBG_RX: now also J3.3 (Pin_3), U3.43 (P0.21); no longer J3.1 (Pin_1), U3.44 (P0.20)
- net DBG_TX: now also J3.1 (Pin_1), U3.44 (P0.20); no longer J3.3 (Pin_3), U3.43 (P0.21)
Changed lines of the file:
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@@
-		)
-	)
-	(label "DBG_TX"
-		(at 140.97 140.97 180)
-		(effects
-			(font
-				(size 1.27 1.27)
-			)
-			(justify right bottom)
 		)
 	)
@@
 		)
 	)
+	(label "DBG_RX"
+		(at 240.03 43.18 180)
+		(effects
+			(font
+				(size 1.27 1.27)
+			)
+			(justify right bottom)
+		)
+	)
 	(label "P4_LED"
 		(at 275.59 97.79 180)
@@
 		)
 	)
+	(label "DBG_RX"
+		(at 140.97 140.97 180)
+		(effects
+			(font
+				(size 1.27 1.27)
+			)
+			(justify right bottom)
+		)
+	)
 	(label "P2_LED"
 		(at 275.59 80.01 180)
@@
 		)
 	)
-	(label "DBG_RX"
+	(label "DBG_TX"
 		(at 240.03 48.26 180)
 		(effects
@@
 		)
 	)
-	(label "DBG_TX"
-		(at 240.03 43.18 180)
-		(effects
-			(font
-				(size 1.27 1.27)
-			)
-			(justify right bottom)
-		)
-	)
 	(label "SWCLK"
 		(at 82.55 97.79 0)
@@
 		)
 	)
-	(label "DBG_RX"
-		(at 140.97 138.43 180)
-		(effects
-			(font
-				(size 1.27 1.27)
-			)
-			(justify right bottom)
-		)
-	)
 	(label "D-"
 		(at 86.36 135.89 0)
@@
 		)
 	)
+	(label "DBG_TX"
+		(at 140.97 138.43 180)
+		(effects
+			(font
+				(size 1.27 1.27)
+			)
+			(justify right bottom)
+		)
+	)
